File: Hardware/Magnetic-Encoder-RS485.kicad_sch (KiCad schematic)
At the start: 32 parts, among them J1 Conn_01x04, J2 Conn_01x04, U1 STM8S003F3P, U2 SP3485EN, U3 MT6816CT-ACD, U4 HT75R33-1A, Y1 X1E0000210119

Commit message: Design is almost done
Parts:
- removed H1, H2, H3, H4: MountingHole_Pad, MountingHole:MountingHole_3.2mm_M3_Pad_Via, symbol Mechanical:MountingHole_Pad
- added D2: LED, LED_SMD:LED_1206_3216Metric_ReverseMount_Hole1.8x2.4mm, symbol Device:LED
- added R2: 100, Resistor_SMD:R_0805_2012Metric, symbol Device:R_Small
- J1: footprint Connector_PinHeader_2.54mm:PinHeader_1x04_P2.54mm_Vertical -> Connector_JST:JST_PH_S4B-PH-K_1x04_P2.00mm_Horizontal; LCSC Part Number (none) -> C157926
- J2: LCSC Part Number (none) -> C160334
Connections:
- net +3V3: now also R2.1
- net +5V: now also J1.4 (Pin_4); no longer J1.1 (Pin_1)
- net A: now also J1.3 (Pin_3); no longer J1.2 (Pin_2)
- net B: now also J1.2 (Pin_2); no longer J1.3 (Pin_3)
- net GND: now also J1.1 (Pin_1), D2.1 (K); no longer J1.4 (Pin_4)
- new net: D2.2 (A), R2.2
- no-connect marks 11 -> 7
Other:
- note removed: "Mounting Holes"
- title: (none) -> Magnetic Encoder RS485
- moved on the sheet: C1, C11, C12, C2, C3, C4, C5, C6, C7, C8, D1, J1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
