File: Hardware/EncoderRS.kicad_sch (KiCad schematic)
At the start: 30 parts, among them J1 Conn_01x04, J2 Conn_01x04, U1 STM8S003F3P, U2 SP3485EN, U3 MT6816CT-ACD, U4 HT75R33-1A, Y1 X1E0000210119

Commit message: Project renamed to EncodeRS
Other:
- title: Magnetic Encoder RS485 -> EncodeRS

Commit message: Updated libs
Parts:
- D2: footprint LED_SMD:LED_1206_3216Metric_ReverseMount_Hole1.8x2.4mm -> encoders_lib:LED_1206_3216Metric_ReverseMount_Hole2.1mm
- U4: symbol Regulator_Linear:HT75xx-1-SOT89 -> encoders_lib:HT75R33-1A
Changed lines of the file:
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@@
 			)
 		)
-		(property "Footprint" "LED_SMD:LED_1206_3216Metric_ReverseMount_Hole1.8x2.4mm"
+		(property "Footprint" "encoders_lib:LED_1206_3216Metric_ReverseMount_Hole2.1mm"
 			(at 140.97 142.24 0)
 			(effects
@@
 	)
 	(symbol
-		(lib_id "Regulator_Linear:HT75xx-1-SOT89")
+		(lib_id "encoders_lib:HT75R33-1A")
 		(at 111.76 135.89 0)
 		(unit 1)
